File: schematic/esp32-switch.kicad_pcb (KiCad board)
At the start: 2 copper layers, 80 x 100 mm, 24 parts, among them J1 Direction, J11 Bouton 5v, J17 Bouton Batterie, J2 + - home, J3 a b x y, J4 L R ZL ZR, J5 Joy D, J6 Joy G, U1 ESP32-DevKitC

Commit message: mise à jour du schema
Parts:
- added D1: 1N4007, Diode_THT:D_DO-41_SOD81_P10.16mm_Horizontal, F.Cu at (153.0, 88.1)
- added J7: Moteur vibration, Connector_AMASS:AMASS_XT30U-F_1x02_P5.0mm_Vertical, F.Cu at (147.0, 81.0)
- added Q1: BC547, Package_TO_SOT_THT:TO-92_Inline, F.Cu at (138.0, 91.0)
- added R3: 1K, Resistor_THT:R_Axial_DIN0204_L3.6mm_D1.6mm_P5.08mm_Vertical, F.Cu at (197.5, 127.0)
- R1, R2: value R -> 10K
- moved J11 7.00 mm to (140.0, 81.0)
- moved Bat+ 2.00 mm to (133.0, 92.0)
- moved Bat- 2.00 mm to (133.0, 97.0)
- moved J17 2.00 mm to (133.0, 81.0)
- moved JP1 0.54 mm to (202.5, 96.0)
- moved JP2 0.54 mm to (202.5, 98.0)
- moved JP3 0.54 mm to (202.5, 93.0)
- moved JP5 0.54 mm to (202.5, 90.0)
- moved JP4 0.21 mm to (202.5, 77.5)
Connections:
- U1 pad 26: unconnected-(U1-ADC2_CH0/GPIO4-Pad26) -> Net-(U1-ADC2_CH0/GPIO4)
Routing:
- net Net-(U1-ADC2_CH0/GPIO4): track 0.00 -> 102.8 mm, vias 0 -> 2
- net Net-(Q1-B): track 0.00 -> 80.6 mm
- net Net-(D1-A): track 0.00 -> 40.2 mm
- net Net-(J1-Pin_2): track 330.4 -> 308.6 mm
- net Net-(D1-K): track 28.2 -> 42.8 mm
- net Net-(J17-Pin_1): track 79.5 -> 84.1 mm
- net Net-(J11-Pin_1): track 36.2 -> 39.1 mm
- net Net-(U1-SENSOR_VP/GPIO36/ADC1_CH0): track 59.5 -> 57.9 mm
- net Net-(JP5-A): track 47.9 -> 47.4 mm
- net Net-(JP3-A): track 48.1 -> 47.6 mm
- net Net-(JP2-A): track 44.7 -> 44.2 mm
- net Net-(JP1-A): track 47.7 -> 47.2 mm
